File: pcb/DidplayAdapter_DOGS104.sch (KiCad schematic (older format))
At the start: 8 parts, among them J1 EA_DOGS104, J2 Amber, U1 EA_DOGS104x-A

Commit message: Uknown changes to merge with master
Parts:
- removed J1: EA_DOGS104, Pin_Headers:Pin_Header_Straight_1x07_Pitch2.54mm, symbol Conn_01x07_Male
- removed J2: Amber, DisplayAdapter_DOGS104_Footprints:Jumper_2_pad, symbol GS2
- added J?: Conn_01x07_Male, symbol Connector:Conn_01x07_Male
- added JP?: SolderJumper_2_Open, symbol Jumper:SolderJumper_2_Open
- C1, C2: symbol C -> Device:C
- R1, R2, R3: symbol R -> Device:R
- U1: symbol EA_DOGS104x-A -> DisplayAdapter_DOGS104_symbols:EA_DOGS104x-A
Connections:
- wire segments 43 -> 52
